Commit message: Add marker on cobod + clean

File: src/cobod_arm/urdf/cobod_arm.urdf (robot description, URDF)
Before this commit: robot cobod_arm, 9 links, 8 joints
Links:
- removed link Gripper_1
- removed link Gripper_2
- link Link_1: mass 4.7914 -> None
Joints:
- removed joint Joint_7
- removed joint Joint_8
