Commit message: trac_ik in function

File: src/cobod_arm_study/urdf/cobod_arm.urdf (robot description, URDF)
Before this commit: robot cobod_arm, 7 links, 6 joints
Links:
- link Gripper_base: geometry collision mesh filename=package://cobod_arm_study/meshes/Gripper_base.STL; visual mesh filename=package://cobod_arm_study/meshes/Gripper_base.STL
- link Link_1: geometry collision mesh filename=package://cobod_arm_study/meshes/Link_1.STL; visual mesh filename=package://cobod_arm_study/meshes/Link_1.STL
- link Link_2: geometry collision mesh filename=package://cobod_arm_study/meshes/Link_2.STL; visual mesh filename=package://cobod_arm_study/meshes/Link_2.STL
- link Link_3: geometry collision mesh filename=package://cobod_arm_study/meshes/Link_3.STL; visual mesh filename=package://cobod_arm_study/meshes/Link_3.STL
- link Link_4: geometry collision mesh filename=package://cobod_arm_study/meshes/Link_4.STL; visual mesh filename=package://cobod_arm_study/meshes/Link_4.STL
- link Link_5: geometry collision mesh filename=package://cobod_arm_study/meshes/Link_5.STL; visual mesh filename=package://cobod_arm_study/meshes/Link_5.STL
- link Link_6: geometry collision mesh filename=package://cobod_arm_study/meshes/Link_6.STL; visual mesh filename=package://cobod_arm_study/meshes/Link_6.STL

Commit message: All clean

File: src/cobod_arm_study/urdf/cobod_arm.urdf (robot description, URDF)
Before this commit: robot cobod_arm_study, 7 links, 6 joints
Links:
- link Gripper_base: geometry collision mesh filename=package://cobod_arm_study/meshes/cobod_arm/Gripper_base.STL; visual mesh filename=package://cobod_arm_study/meshes/cobod_arm/Gripper_base.STL
- link Link_1: geometry collision mesh filename=package://cobod_arm_study/meshes/cobod_arm/Link_1.STL; visual mesh filename=package://cobod_arm_study/meshes/cobod_arm/Link_1.STL
- link Link_2: geometry collision mesh filename=package://cobod_arm_study/meshes/cobod_arm/Link_2.STL; visual mesh filename=package://cobod_arm_study/meshes/cobod_arm/Link_2.STL
- link Link_3: geometry collision mesh filename=package://cobod_arm_study/meshes/cobod_arm/Link_3.STL; visual mesh filename=package://cobod_arm_study/meshes/cobod_arm/Link_3.STL
- link Link_4: geometry collision mesh filename=package://cobod_arm_study/meshes/cobod_arm/Link_4.STL; visual mesh filename=package://cobod_arm_study/meshes/cobod_arm/Link_4.STL
- link Link_5: geometry collision mesh filename=package://cobod_arm_study/meshes/cobod_arm/Link_5.STL; visual mesh filename=package://cobod_arm_study/meshes/cobod_arm/Link_5.STL
- link Link_6: geometry collision mesh filename=package://cobod_arm_study/meshes/cobod_arm/Link_6.STL; visual mesh filename=package://cobod_arm_study/meshes/cobod_arm/Link_6.STL

Commit message: update joint limit urdf cobot

File: src/cobod_arm_study/urdf/cobod_arm.urdf (robot description, URDF)
Before this commit: robot cobod_arm_study, 7 links, 6 joints
Joints:
- joint Joint_2: limit lower=-1.5707963268 upper=1.5707963268 effort=10 velocity=1.0 -> lower=-1.5707963268 upper=0.62 effort=10 velocity=1.0
- joint Joint_3: limit lower=-1.5707963268 upper=1.5707963268 effort=8 velocity=1.0 -> lower=0.0 upper=1.5707963268 effort=8 velocity=1.0
- joint Joint_5: limit lower=-1.5707963268 upper=1.5707963268 effort=6 velocity=1.0 -> lower=-1.5707963268 upper=0.0 effort=6 velocity=1.0
